Commit message: real robot configs

File: nav2_minimal_description/urdf/sensors/rplidar.urdf.xacro (robot description, xacro)
@@ -12,8 +12,8 @@
   <joint name="${name}_joint" type="fixed">
     <parent link="${parent_link}"/>
-    <child link="${name}_link"/>
+    <child link="${name}"/>
     <xacro:insert_block name="origin"/>
   </joint>
-  <link name="${name}_link">
+  <link name="${name}">
     <visual>
       <geometry>
@@ -29,5 +29,5 @@
     <xacro:inertial_cuboid mass="0.17" x="${length_x}" y="${length_y}" z="${length_z}"/>
   </link>
-  <gazebo reference="${name}_link">
+  <gazebo reference="${name}">
     <xacro:ray_sensor sensor_name="${name}" gazebo="${gazebo}"
                   update_rate="10.0" visualize="true"

File: nav2_minimal_description/urdf/standard/turtlebot4.urdf.xacro (robot description, xacro)
@@ -108,6 +108,6 @@
   </xacro:tower_sensor_plate>
   <!-- Turtlebot4 sensor definitions -->
-  <xacro:rplidar name="rplidar" parent_link="shell_link" gazebo="$(arg gazebo)">
-    <origin xyz="${rplidar_x_offset} ${rplidar_y_offset} ${rplidar_z_offset}" rpy="0 0 ${pi/2}"/>
+  <xacro:rplidar name="base_laser" parent_link="shell_link" gazebo="$(arg gazebo)">
+    <origin xyz="${rplidar_x_offset} ${rplidar_y_offset} ${rplidar_z_offset}" rpy="0 0 -${pi/2}"/>
   </xacro:rplidar>
   <xacro:camera_bracket name="oakd_camera_bracket">

File: test_tb4.urdf (robot description, URDF)
Before this commit: robot turtlebot4, 32 links, 31 joints
Links:
- removed link rplidar_link
- added link base_laser, mass 0.17; collision box size=0.071 0.1 0.06; visual mesh filename=package://nav2_minimal_description/meshes/rplidar.dae scale=1 1 1
Joints:
- joint rplidar_joint: child rplidar_link -> base_laser; origin xyz=-0.04 0.0 0.098715 rpy=0 0 1.5707963267948966 -> xyz=-0.04 0.0 0.098715 rpy=0 0 0
